File: pcb/MCU.kicad_sch (KiCad schematic)
At the start: 11 parts, among them U301 WeMos_S2_mini

Commit message: revision 2.0: changed R and C footprints to 0805 (imperial)
Parts:
- R301, R302, R303: footprint Resistor_SMD:R_0603_1608Metric -> Resistor_SMD:R_0805_2012Metric
Changed lines of the file:
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@@
 			)
 		)
-		(property "Footprint" "Resistor_SMD:R_0603_1608Metric"
+		(property "Footprint" "Resistor_SMD:R_0805_2012Metric"
 			(at 227.33 47.498 90)
 			(effects
@@
 			)
 		)
-		(property "Footprint" "Resistor_SMD:R_0603_1608Metric"
+		(property "Footprint" "Resistor_SMD:R_0805_2012Metric"
 			(at 227.33 52.578 90)
 			(effects
@@
 			)
 		)
-		(property "Footprint" "Resistor_SMD:R_0603_1608Metric"
+		(property "Footprint" "Resistor_SMD:R_0805_2012Metric"
 			(at 227.33 57.658 90)
 			(effects

Commit message: components updates
Parts:
- R301, R302, R303: value 180 -> 200
Changed lines of the file:
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@@
 			)
 		)
-		(property "Value" "180"
+		(property "Value" "200"
 			(at 227.076 48.26 90)
 			(effects
@@
 			)
 		)
-		(property "Value" "180"
+		(property "Value" "200"
 			(at 227.076 53.34 90)
 			(effects
@@
 			)
 		)
-		(property "Value" "180"
+		(property "Value" "200"
 			(at 227.33 58.42 90)
 			(effects
